File: hardware/rsr232-iso/rsr232-iso.kicad_sch (KiCad schematic)
At the start: 16 parts, among them J1 Serial, J2 PWR, J3 data, U1 MAX3232, U2 TLP2358, U3 TLP2358

Commit message: Use a 2DIB1411F isolator instead of 2 optocouplers
Parts:
- removed R1: 330, Resistor_SMD:R_0805_2012Metric_Pad1.20x1.40mm_HandSolder, symbol Device:R_Small
- removed R2: 220, Resistor_SMD:R_0805_2012Metric_Pad1.20x1.40mm_HandSolder, symbol Device:R_Small
- removed U2, U3: TLP2358, Package_SO:SO-6L_10x3.84mm_P1.27mm, symbol Isolator:TLP2748
- added C8: 100nF, Capacitor_SMD:C_0603_1608Metric_Pad1.08x0.95mm_HandSolder, symbol Device:C_Small
- added H1: MountingHole, MountingHole:MountingHole_3.2mm_M3_DIN965, symbol Mechanical:MountingHole
- added U2: ADuM1201AR, Package_SO:SOIC-8_3.9x4.9mm_P1.27mm, symbol Isolator:ADuM1201AR
Connections:
- net +3.3V: now also U2.1 (VDD1)
- net +5V: now also C8.1, U2.8 (VDD2)
- net GND: now also C8.2, U2.5 (GND2)
- net GNDD: now also U2.4 (GND1)
- net RX: now also J3.2 (Pin_2), U2.2 (VOA); no longer J3.1 (Pin_1)
- net TX: now also J3.1 (Pin_1), U2.3 (VIB); no longer J3.2 (Pin_2)
- net at U1.9 (R2OUT): now also U2.7 (VIA)
- net at U1.10 (T2IN): now also U2.6 (VOB)
Other:
- moved on the sheet: J3

Commit message: Correct isolator reference
Parts:
- U2: value ADuM1201AR -> 2DIB1411F; P/N (none) -> 2DIB1411F
Changed lines of the file:
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@@
 			)
 		)
-		(property "Value" "ADuM1201AR"
+		(property "Value" "2DIB1411F"
 			(at 93.98 94.7998 0)
 			(effects
@@
 			)
 		)
-		(property "Datasheet" "https://www.analog.com/media/en/technical-documentation/data-sheets/ADuM1200_1201.pdf"
+		(property "Datasheet" ""
 			(at 93.98 106.68 0)
 			(effects
@@
 			(at 93.98 104.14 0)
 			(effects
+				(font
+					(size 1.27 1.27)
+				)
+				(hide yes)
+			)
+		)
+		(property "P/N" "2DIB1411F"
+			(at 93.98 104.14 0)
+			(effects
