File: hardware/energie/energie.kicad_sch (KiCad schematic)
At the start: 55 parts, among them J1 transfos, J2 Conn_01x05_Pin, J3 linky, J4 Serial, J6 gpio, J7 I2C, J8 power, J9 ACin, Q1 BSS123, Q2 BSS123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

Commit message: energie: name rs232_RX/TX
Connections:
- net rs232_TX: now reaches J4.1 (Pin_1), U4.7 (T2OUT)
- net rs232_RX: now reaches J4.2 (Pin_2), U4.8 (R2IN)
Changed lines of the file:
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@@
+		)
+	)
+	(label "rs232_RX"
+		(at 219.71 80.01 0)
+		(fields_autoplaced yes)
+		(effects
+			(font
+				(size 1.27 1.27)
+			)
+			(justify left bottom)
+		)
+	)
+	(label "rs232_TX"
+		(at 219.71 69.85 0)
+		(fields_autoplaced yes)
+		(effects
+			(font
+				(size 1.27 1.27)
+			)
+			(justify left bottom)
 		)
 	)
