File: hardware/ventil/ventil.kicad_pcb (KiCad board)
At the start: 2 copper layers, 60 x 42 mm, 32 parts, among them J1 Conn_01x05_Pin, J2 M, J3 BUS, J4 i2C, Q1 BSS123, U1 SHT31-DIS, U2 PIC18F05Q40, U4 MCP2003B, U5 uA7805, U6 ULN2003

Commit message: ventil, vmc: switch 7805 to a less expensive package
Parts:
- U5: footprint Package_TO_SOT_SMD:SOT-223-3_TabPin2 -> Package_TO_SOT_SMD:TO-252-3_TabPin2
- moved C9 2.79 mm to (138.8, 118.4), turned to 90 degrees
- moved C5 1.42 mm to (143.1, 122.2)
Routing:
- net GND: track 110.8 -> 108.8 mm
- net +12V: track 145.5 -> 147.1 mm
- net +5V: track 118.2 -> 116.7 mm
