File: hardware/ventil/ventil.kicad_pcb (KiCad board)
At the start: 2 copper layers, 60 x 42 mm, 32 parts, among them J1 Conn_01x05_Pin, J2 M, J3 BUS, J4 i2C, Q1 BSS123, U1 SHT31-DIS, U2 PIC18F05Q40, U4 MCP2003B, U5 uA7805, U6 ULN2003

Commit message: hardware/ventil: name SCL/SDA
Connections:
- net Net-(J4-Pin_3) renamed /SCL
- net Net-(J4-Pin_4) renamed /SDA
Changed lines of the file:
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@@
 	(net 13 "unconnected-(J3-Pin_2-Pad2)")
 	(net 14 "unconnected-(J3-Pin_2-Pad2)_1")
-	(net 15 "Net-(J4-Pin_4)")
-	(net 16 "Net-(J4-Pin_3)")
+	(net 15 "/SDA")
+	(net 16 "/SCL")
 	(net 17 "/LED")
 	(net 18 "Net-(U4-~{WAKE})")
@@
 			(layers "F.Cu" "F.Paste" "F.Mask")
 			(roundrect_rratio 0.208333)
-			(net 16 "Net-(J4-Pin_3)")
+			(net 16 "/SCL")
 			(pintype "passive")
 		)
@@
 			(layers "F.Cu" "F.Paste" "F.Mask")
 			(roundrect_rratio 0.25)
-			(net 16 "Net-(J4-Pin_3)")
+			(net 16 "/SCL")
 			(pinfunction "RC1/CxIN1-/SDA")
 			(pintype "bidirectional")
@@
 			(layers "F.Cu" "F.Paste" "F.Mask")
 			(roundrect_rratio 0.25)
-			(net 15 "Net-(J4-Pin_4)")
+			(net 15 "/SDA")
 			(pinfunction "RC0/C2IN0+/SCL")
 			(pintype "bidirectional")
@@
 			(size 0.55 0.25)
 			(layers "F.Cu" "F.Paste" "F.Mask")
-			(net 15 "Net-(J4-Pin_4)")
+			(net 15 "/SDA")
 			(pinfunction "SDA")
 			(pintype "bidirectional")
@@
 			(size 0.55 0.25)
 			(layers "F.Cu" "F.Paste" "F.Mask")
-			(net 16 "Net-(J4-Pin_3)")
+			(net 16 "/SCL")
 			(pinfunction "SCL")
 			(pintype "input")
@@
 			(layers "F.Cu" "F.Paste" "F.Mask")
 			(roundrect_rratio 0.208333)
-			(net 15 "Net-(J4-Pin_4)")
+			(net 15 "/SDA")
 			(pintype "passive")
 		)
@@
 			(layers "F.Cu" "F.Paste" "F.Mask")
 			(roundrect_rratio 0.25)
-			(net 16 "Net-(J4-Pin_3)")
+			(net 16 "/SCL")
 			(pinfunction "Pin_3")
 			(pintype "passive")
@@
 			(layers "F.Cu" "F.Paste" "F.Mask")
 			(roundrect_rratio 0.25)
-			(net 16 "Net-(J4-Pin_3)")
+			(net 16 "/SCL")
 			(pinfunction "Pin_3")
 			(pintype "passive")
@@
 			(layers "F.Cu" "F.Paste" "F.Mask")
 			(roundrect_rratio 0.25)
-			(net 15 "Net-(J4-Pin_4)")
+			(net 15 "/SDA")
 			(pinfunction "Pin_4")
 			(pintype "passive")
@@
 			(layers "F.Cu" "F.Paste" "F.Mask")
 			(roundrect_rratio 0.25)
-			(net 15 "Net-(J4-Pin_4)")
+			(net 15 "/SDA")
 			(pinfunction "Pin_4")
 			(pintype "passive")
