File: hardware/ventil/ventil.kicad_sch (KiCad schematic)
At the start: 28 parts, among them J1 Conn_01x05_Pin, J2 M, J3 BUS, J4 i2C, Q1 BSS123, U1 SHT31-DIS, U2 PIC18F05Q40, U4 MCP2003B, U5 uA7805, U6 ULN2003

Commit message: ventil: route PCB
Parts:
- added H1, H2, H3, H4: MountingHole, MountingHole:MountingHole_3.2mm_M3, symbol Mechanical:MountingHole
Connections:
- net +12V: now also J2.1 (Pin_1); no longer J2.5 (Pin_5)
- net +5V: now also J1.2 (Pin_2); no longer J1.5 (Pin_5)
- net GND: now also J1.3 (Pin_3); no longer J1.2 (Pin_2)
- net PGC: now also J1.5 (Pin_5); no longer J1.3 (Pin_3)
- net at R3.1, U1.4 (SCL), U2.9 (RC1/CxIN1-/SDA): now also J4.3 (Pin_3); no longer J4.4 (Pin_4)
- net at U6.13 (O4): now also J2.5 (Pin_5); no longer J2.1 (Pin_1)
- net at U6.14 (O3): now also J2.4 (Pin_4); no longer J2.2 (Pin_2)
- net at U6.16 (O1): now also J2.2 (Pin_2); no longer J2.4 (Pin_4)
- net at R2.1, U1.1 (SDA), U2.10 (RC0/C2IN0+/SCL): now also J4.4 (Pin_4); no longer J4.3 (Pin_3)
Other:
- moved on the sheet: J4, R6

Commit message: ventil, vmc: switch 7805 to a less expensive package
Parts:
- U5: footprint Package_TO_SOT_SMD:SOT-223-3_TabPin2 -> Package_TO_SOT_SMD:TO-252-3_TabPin2
Changed lines of the file:
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@@
 			)
 		)
-		(property "Footprint" "Package_TO_SOT_SMD:SOT-223-3_TabPin2"
+		(property "Footprint" "Package_TO_SOT_SMD:TO-252-3_TabPin2"
 			(at 98.425 167.64 0)
 			(effects
