File: hardware/controle/controle.kicad_pcb (KiCad board)
At the start: 2 copper layers, 83.6 x 76.7 mm, 94 parts, among them J1 TWI3, J10 Conn_01x05_Pin, J11 ADC, J12 PWM, J2 SENS0375, J3 TWI4, J4 LED, J5 UART7, J6 PWR, J7 DATA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

Commit message: hardware/controle: update P/N fields
Parts:
- D7: value Red -> RED
Changed lines of the file:
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@@
 			)
 		)
-		(property "P/N" "stock"
+		(property "P/N" "MCWR08X2201FTL"
 			(at 0 0 180)
 			(unlocked yes)
@@
 			)
 		)
-		(property "P/N" "CL21A475KPFNNNE"
+		(property "P/N" "08053C475KAT2A"
 			(at 0 0 180)
 			(unlocked yes)
@@
 			)
 		)
-		(property "P/N" "C3225X5R1E106K250AA (stock)"
+		(property "P/N" "GRM21BC8YA106KE11L"
 			(at 0 0 180)
 			(unlocked yes)
@@
 			)
 		)
-		(property "P/N" "stock"
+		(property "P/N" "MCWR08X5602FTL"
 			(at 0 0 0)
 			(unlocked yes)
@@
 			)
 		)
-		(property "P/N" "CGA3E1X7R1V105K080AC (stock)"
+		(property "P/N" "CGA3E1X7R1V105K080AC"
 			(at 0 0 180)
 			(unlocked yes)
@@
 			)
 		)
-		(property "P/N" "stock"
+		(property "P/N" "MCWR08X2201FTL"
 			(at 0 0 180)
 			(unlocked yes)
@@
 			)
 		)
-		(property "P/N" "stock"
+		(property "P/N" "MCWR08X5602FTL"
 			(at 0 0 180)
 			(unlocked yes)
@@
 			)
 		)
-		(property "P/N" "C0805C105K3RACTU ou 08053C105KAT9A (stock)"
+		(property "P/N" "C0805C105K3RACTU ou 08053C105KAT9A"
 			(at 0 0 0)
 			(unlocked yes)
@@
 			)
 		)
-		(property "P/N" "stock"
+		(property "P/N" "MCWR08X5602FTL"
 			(at 0 0 180)
 			(unlocked yes)
@@
 			)
 		)
-		(property "P/N" "C3225X5R1E106K250AA (stock)"
+		(property "P/N" "GRM21BC8YA106KE11L"
 			(at 0 0 180)
 			(unlocked yes)
@@
 			)
 		)
-		(property "P/N" "stock"
+		(property "P/N" "MCWR08X5602FTL"
 			(at 0 0 0)
 			(unlocked yes)
@@
 			)
 		)
-		(property "P/N" "stock"
+		(property "P/N" "MCWR08X1002FTL"
 			(at 0 0 180)
 			(unlocked yes)
@@
 			)
 		)
-		(property "P/N" "C3225X5R1A226M230AA/CL31A226KAHNNN (stock)"
+		(property "P/N" "C3225X5R1A226M230AA/CL31A226KAHNNN"
 			(at 0 0 0)
 			(unlocked yes)
@@
 			)
 		)
-		(property "P/N" "stock"
+		(property "P/N" "MCWR08X1002FTL"
 			(at 0 0 180)
 			(unlocked yes)
@@
 			)
 		)
-		(property "P/N" "C3225X5R1A226M230AA/CL31A226KAHNNN (stock)"
+		(property "P/N" "C3225X5R1A226M230AA/CL31A226KAHNNN"
 			(at 0 0 0)
 			(unlocked yes)
@@
 			)
 		)
-		(property "P/N" "CL21A475KPFNNNE"
+		(property "P/N" "08053C475KAT2A"
 			(at 0 0 0)
 			(unlocked yes)
@@
 			)
 		)
-		(property "P/N" "stock"
+		(property "P/N" "MCWR08X1002FTL"
 			(at 0 0 -90)
 			(unlocked yes)
@@
 			)
 		)
-		(property "P/N" "stock"
+		(property "P/N" "MCWR08X1002FTL"
 			(at 0 0 0)
 			(unlocked yes)
@@
 			)
 		)
-		(property "P/N" "stock"
+		(property "P/N" "MCWR08X5602FTL"
 			(at 0 0 0)
 			(unlocked yes)
@@
 			)
 		)
-		(property "P/N" "GRM188R71H682KA01D (stock)"
+		(property "P/N" "C0603C682K5R"
 			(at 0 0 0)
 			(unlocked yes)
@@
 			)
 		)
-		(property "P/N" "87437-0543"
+		(property "P/N" ""
 			(at 0 0 90)
 			(unlocked yes)
@@
 			)
 		)
-		(property "Value" "Red"
+		(property "Value" "RED"
 			(at 0 -1.65 90)
 			(layer "B.Fab")

Commit message: rdware/controle: move back some resistors to 47k to match our stock
Parts:
- R22, R23, R24, R26: value 56K -> 47K
Changed lines of the file:
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@@
 			)
 		)
-		(property "Value" "56K"
+		(property "Value" "47K"
 			(at 0 1.65 0)
 			(layer "F.Fab")
@@
 			)
 		)
-		(property "P/N" "MCWR08X5602FTL"
+		(property "P/N" "MCWR08X4702FTL"
 			(at 0 0 0)
 			(unlocked yes)
@@
 			)
 		)
-		(property "Value" "56K"
+		(property "Value" "47K"
 			(at 0 1.65 0)
 			(layer "F.Fab")
@@
 			)
 		)
-		(property "P/N" "MCWR08X5602FTL"
+		(property "P/N" "MCWR08X4702FTL"
 			(at 0 0 180)
 			(unlocked yes)
@@
 			)
 		)
-		(property "Value" "56K"
+		(property "Value" "47K"
 			(at 0 1.65 0)
 			(layer "F.Fab")
@@
 			)
 		)
-		(property "P/N" "MCWR08X5602FTL"
+		(property "P/N" "MCWR08X4702FTL"
 			(at 0 0 180)
 			(unlocked yes)
@@
 			)
 		)
-		(property "Value" "56K"
+		(property "Value" "47K"
 			(at 0 1.65 0)
 			(layer "F.Fab")
@@
 			)
 		)
-		(property "P/N" "MCWR08X5602FTL"
+		(property "P/N" "MCWR08X4702FTL"
 			(at 0 0 0)
 			(unlocked yes)
