File: hardware/controle/power.kicad_sch (KiCad schematic)
At the start: 21 parts, among them J9 Barrel_Jack, U4 TPS54228, U5 NCP718xSN330

Commit message: hardware/controle: update P/N of 100nF capacitors
Parts:
- C11: P/N C0603C100J5ACTU -> C0603C100J5GACTU
- C8: P/N CC0805KKX7RYBB104 -> C0603C104K5RAC7411
Changed lines of the file:
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@@
 			)
 		)
-		(property "P/N" "CC0805KKX7RYBB104"
+		(property "P/N" "C0603C104K5RAC7411"
 			(at 179.07 27.94 0)
 			(effects
@@
 			)
 		)
-		(property "P/N" "C0603C100J5ACTU"
+		(property "P/N" "C0603C100J5GACTU"
 			(at 148.59 92.71 0)
 			(effects
